File: CurrentVolt.kicad_sch (KiCad schematic)
At the start: 3 parts, among them U6 ACS70331EOLCTR-2P5U3

Commit message: working on MUX and pre-amp layout
Changed lines of the file:
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@@
 (kicad_sch (version 20211123) (generator eeschema)
   (paper "A4")
+  (junction (at 84.328 96.52) (diameter 0) (color 0 0 0 0)
+  )
   (junction (at 81.28 81.28) (diameter 0) (color 0 0 0 0)
   )
   (junction (at 81.28 67.818) (diameter 0) (color 0 0 0 0)
   )
+  (junction (at 84.582 81.28) (diameter 0) (color 0 0 0 0)
+  )
   (junction (at 78.232 96.52) (diameter 0) (color 0 0 0 0)
   )
@@
     (stroke (width 0) (type default) (color 0 0 0 0))
   )
+  (wire (pts (xy 84.582 81.28) (xy 86.36 81.28))
+    (stroke (width 0) (type default) (color 0 0 0 0))
+  )
   (wire (pts (xy 71.12 96.52) (xy 78.232 96.52))
     (stroke (width 0) (type default) (color 0 0 0 0))
@@
     (stroke (width 0) (type default) (color 0 0 0 0))
   )
-  (wire (pts (xy 78.232 96.52) (xy 86.36 96.52))
+  (wire (pts (xy 78.232 96.52) (xy 84.328 96.52))
     (stroke (width 0) (type default) (color 0 0 0 0))
   )
@@
     (stroke (width 0) (type default) (color 0 0 0 0))
   )
-  (wire (pts (xy 81.28 81.28) (xy 86.36 81.28))
+  (wire (pts (xy 81.28 81.28) (xy 84.582 81.28))
     (stroke (width 0) (type default) (color 0 0 0 0))
   )
@@
   )
   (wire (pts (xy 81.28 81.28) (xy 81.28 83.566))
+    (stroke (width 0) (type default) (color 0 0 0 0))
+  )
+  (wire (pts (xy 84.328 96.52) (xy 86.36 96.52))
     (stroke (width 0) (type default) (color 0 0 0 0))
   )
@@
     (pin "2")
   )
+  (symbol (lib_id "power:PWR_FLAG") (at 84.328 96.52 0) (unit 1)
+    (in_bom yes) (on_board yes) (fields_autoplaced)
+    (property "Reference" "#FLG0105" (id 0) (at 84.328 94.615 0)
+      (effects (font (size 1.27 1.27)) hide)
+    )
+    (property "Value" "PWR_FLAG" (id 1) (at 84.328 91.44 0)
+      (effects (font (size 1.27 1.27)) hide)
+    )
+    (property "Footprint" "" (id 2) (at 84.328 96.52 0)
+      (effects (font (size 1.27 1.27)) hide)
+    )
+    (property "Datasheet" "~" (id 3) (at 84.328 96.52 0)
+      (effects (font (size 1.27 1.27)) hide)
+    )
+    (pin "1")
+  )
   (symbol (lib_id "power:GNDREF") (at 78.232 101.6 0) (unit 1)
     (in_bom yes) (on_board yes) (fields_autoplaced)
@@
       (effects (font (size 1.27 1.27)) hide)
     )
+    (pin "1")
+  )
+  (symbol (lib_id "power:PWR_FLAG") (at 84.582 81.28 0) (unit 1)
+    (in_bom yes) (on_board yes) (fields_autoplaced)
+    (property "Reference" "#FLG0116" (id 0) (at 84.582 79.375 0)
+      (effects (font (size 1.27 1.27)) hide)
+    )
+    (property "Value" "PWR_FLAG" (id 1) (at 84.582 76.2 0)
+      (effects (font (size 1.27 1.27)) hide)
+    )
+    (property "Footprint" "" (id 2) (at 84.582 81.28 0)
+      (effects (font (size 1.27 1.27)) hide)
+    )
+    (property "Datasheet" "~" (id 3) (at 84.582 81.28 0)
+      (effects (font (size 1.27 1.27)) hide)
+    )
