File: dualadj.kicad_sch (KiCad schematic)
At the start: 14 parts, among them J8 Conn_01x02_Female, J9 Conn_01x02_Female, U1 LM317_TO-220, U2 LM337_TO220

Commit message: working on MUX and pre-amp layout
Changed lines of the file:
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@@
     (pin "3")
+  )
+  (symbol (lib_id "power:PWR_FLAG") (at 120.142 72.39 0) (unit 1)
+    (in_bom yes) (on_board yes) (fields_autoplaced)
+    (property "Reference" "#FLG0114" (id 0) (at 120.142 70.485 0)
+      (effects (font (size 1.27 1.27)) hide)
+    )
+    (property "Value" "PWR_FLAG" (id 1) (at 120.142 67.31 0))
+    (property "Footprint" "" (id 2) (at 120.142 72.39 0)
+      (effects (font (size 1.27 1.27)) hide)
+    )
+    (property "Datasheet" "~" (id 3) (at 120.142 72.39 0)
+      (effects (font (size 1.27 1.27)) hide)
+    )
+    (pin "1")
   )
   (symbol (lib_id "minipowersupply-rescue:R_POT_Small-Device") (at 126.492 115.824 0) (unit 1)
@@
     (pin "3")
   )
+  (symbol (lib_id "power:PWR_FLAG") (at 119.888 103.124 0) (unit 1)
+    (in_bom yes) (on_board yes) (fields_autoplaced)
+    (property "Reference" "#FLG0113" (id 0) (at 119.888 101.219 0)
+      (effects (font (size 1.27 1.27)) hide)
+    )
+    (property "Value" "PWR_FLAG" (id 1) (at 119.888 97.79 0))
+    (property "Footprint" "" (id 2) (at 119.888 103.124 0)
+      (effects (font (size 1.27 1.27)) hide)
+    )
+    (property "Datasheet" "~" (id 3) (at 119.888 103.124 0)
+      (effects (font (size 1.27 1.27)) hide)
+    )
+    (pin "1")
+  )
   (symbol (lib_id "Device:FerriteBead_Small") (at 106.172 103.124 90) (unit 1)
